File: EduSat v2/OBCv1/OBCv1.kicad_sch (KiCad schematic)
At the start: 9 parts, among them J1 Conn_02x20_Odd_Even, J2 USB_C_Receptacle_USB2.0_16P, U1 ESP32-WROOM-32E, U2 CP2102N-Axx-xQFN28

Commit message: Another upload
Parts:
- added U3: Ai-Thinker-Ra-02, RF_Module:Ai-Thinker-Ra-01-LoRa, symbol RF_Module:Ai-Thinker-Ra-02
Connections:
- new net: U3.1 (GND), U3.16 (GND), U3.2 (GND), U3.9 (GND)
Other:
- moved on the sheet: H1, H2, H3, H4, J1, U1, U2
Changed lines of the file:
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@@
 	(symbol
 		(lib_id "Mechanical:MountingHole")
-		(at 162.56 96.52 0)
+		(at 133.35 176.53 0)
 		(unit 1)
 		(exclude_from_sim no)
@@
 		(fields_autoplaced yes)
 		(property "Reference" "H2"
-			(at 165.1 95.2499 0)
+			(at 135.89 175.2599 0)
 			(effects
 				(font
@@
 		)
 		(property "Value" "MountingHole"
-			(at 165.1 97.7899 0)
+			(at 135.89 177.7999 0)
 			(effects
 				(font
@@
 		)
 		(property "Footprint" "MountingHole:MountingHole_3.2mm_M3"
-			(at 162.56 96.52 0)
+			(at 133.35 176.53 0)
 			(effects
 				(font
@@
 		)
 		(property "Datasheet" "~"
-			(at 162.56 96.52 0)
+			(at 133.35 176.53 0)
 			(effects
 				(font
@@
 		)
 		(property "Description" "Mounting Hole without connection"
-			(at 162.56 96.52 0)
+			(at 133.35 176.53 0)
 			(effects
 				(font
@@
 	(symbol
 		(lib_id "Mechanical:MountingHole")
-		(at 162.56 111.76 0)
+		(at 133.35 191.77 0)
 		(unit 1)
 		(exclude_from_sim no)
@@
 		(fields_autoplaced yes)
 		(property "Reference" "H4"
-			(at 165.1 110.4899 0)
+			(at 135.89 190.4999 0)
 			(effects
 				(font
@@
 		)
 		(property "Value" "MountingHole"
-			(at 165.1 113.0299 0)
+			(at 135.89 193.0399 0)
 			(effects
 				(font
@@
 		)
 		(property "Footprint" "MountingHole:MountingHole_3.2mm_M3"
-			(at 162.56 111.76 0)
+			(at 133.35 191.77 0)
 			(effects
 				(font
@@
 		)
 		(property "Datasheet" "~"
-			(at 162.56 111.76 0)
+			(at 133.35 191.77 0)
 			(effects
 				(font
@@
 		)
 		(property "Description" "Mounting Hole without connection"
-			(at 162.56 111.76 0)
+			(at 133.35 191.77 0)
 			(effects
 				(font
@@
 	(symbol
 		(lib_id "Connector_Generic:Conn_02x20_Odd_Even")
-		(at 133.35 99.06 0)
+		(at 162.56 31.75 90)
 		(unit 1)
 		(exclude_from_sim no)
@@
 		(fields_autoplaced yes)
 		(property "Reference" "J1"
-			(at 134.62 69.85 0)
-			(effects
-				(font
-					(size 1.27 1.27)
-				)
+			(at 137.16 29.2099 90)
+			(effects
+				(font
+					(size 1.27 1.27)
+				)
+				(justify left)
 			)
 		)
 		(property "Value" "Conn_02x20_Odd_Even"
-			(at 134.62 72.39 0)
-			(effects
-				(font
-					(size 1.27 1.27)
-				)
+			(at 137.16 31.7499 90)
+			(effects
+				(font
+					(size 1.27 1.27)
+				)
+				(justify left)
 			)
 		)
 		(property "Footprint" "Connector_PinSocket_2.54mm:PinSocket_2x20_P2.54mm_Vertical"
-			(at 133.35 99.06 0)
+			(at 162.56 31.75 0)
 			(effects
 				(font
@@
 		)
 		(property "Datasheet" "~"
-			(at 133.35 99.06 0)
+			(at 162.56 31.75 0)
 			(effects
 				(font
@@
 		)
 		(property "Description" "Generic connector, double row, 02x20, odd/even pin numbering scheme (row 1 odd numbers, row 2 even numbers), script generated (kicad-library-utils/schlib/autogen/connector/)"
-			(at 133.35 99.06 0)
+			(at 162.56 31.75 0)
 			(effects
 				(font
@@
 	(symbol
 		(lib_id "Mechanical:MountingHole")
-		(at 162.56 88.9 0)
+		(at 133.35 168.91 0)
 		(unit 1)
 		(exclude_from_sim no)
@@
 		(fields_autoplaced yes)
 		(property "Reference" "H1"
-			(at 165.1 87.6299 0)
+			(at 135.89 167.6399 0)
 			(effects
 				(font
@@
 		)
 		(property "Value" "MountingHole"
-			(at 165.1 90.1699 0)
+			(at 135.89 170.1799 0)
 			(effects
 				(font
@@
 		)
 		(property "Footprint" "MountingHole:MountingHole_3.2mm_M3"
-			(at 162.56 88.9 0)
+			(at 133.35 168.91 0)
 			(effects
 				(font
@@
 		)
 		(property "Datasheet" "~"
-			(at 162.56 88.9 0)
+			(at 133.35 168.91 0)
 			(effects
 				(font
@@
 		)
 		(property "Description" "Mounting Hole without connection"
-			(at 162.56 88.9 0)
+			(at 133.35 168.91 0)
 			(effects
 				(font
@@
 	(symbol
 		(lib_id "Interface_USB:CP2102N-Axx-xQFN28")
-		(at 220.98 91.44 0)
+		(at 223.52 99.06 0)
+		(mirror y)
 		(unit 1)
 		(exclude_from_sim no)
@@
 		(on_board yes)
 		(dnp no)
-		(fields_autoplaced yes)
 		(property "Reference" "U2"
-			(at 223.1741 124.46 0)
+			(at 221.3259 132.08 0)
 			(effects
 				(font
@@
 		)
 		(property "Value" "CP2102N-Axx-xQFN28"
-			(at 223.1741 127 0)
+			(at 221.3259 134.62 0)
 			(effects
 				(font
@@
 		)
 		(property "Footprint" "Package_DFN_QFN:QFN-28-1EP_5x5mm_P0.5mm_EP3.35x3.35mm"
-			(at 254 123.19 0)
+			(at 190.5 130.81 0)
 			(effects
 				(font
@@
 		)
 		(property "Datasheet" "https://www.silabs.com/documents/public/data-sheets/cp2102n-datasheet.pdf"
-			(at 222.25 110.49 0)
+			(at 222.25 118.11 0)
 			(effects
 				(font
@@
 		)
 		(property "Description" "USB to UART master bridge, QFN-28"
-			(at 220.98 91.44 0)
+			(at 223.52 99.06 0)
 			(effects
 				(font
@@
 	(symbol
 		(lib_id "RF_Module:ESP32-WROOM-32E")
-		(at 92.71 91.44 0)
+		(at 106.68 86.36 0)
 		(unit 1)
 		(exclude_from_sim no)
@@
 		(fields_autoplaced yes)
 		(property "Reference" "U1"
-			(at 94.9041 53.34 0)
+			(at 108.8741 48.26 0)
 			(effects
 				(font
@@
 		)
 		(property "Value" "ESP32-WROOM-32E"
-			(at 94.9041 55.88 0)
+			(at 108.8741 50.8 0)
 			(effects
 				(font
@@
 		)
 		(property "Footprint" "RF_Module:ESP32-WROOM-32D"
-			(at 109.22 125.73 0)
+			(at 123.19 120.65 0)
 			(effects
 				(font
@@
 		)
 		(property "Datasheet" "https://www.espressif.com/sites/default/files/documentation/esp32-wroom-32e_esp32-wroom-32ue_datasheet_en.pdf"
-			(at 92.71 91.44 0)
+			(at 106.68 86.36 0)
 			(effects
 				(font
@@
 		)
 		(property "Description" "RF Module, ESP32-D0WD-V3 SoC, without PSRAM, Wi-Fi 802.11b/g/n, Bluetooth, BLE, 32-bit, 2.7-3.6V, onboard antenna, SMD"
-			(at 92.71 91.44 0)
+			(at 106.68 86.36 0)
 			(effects
 				(font
@@
 	(symbol
 		(lib_id "Mechanical:MountingHole")
-		(at 162.56 104.14 0)
+		(at 133.35 184.15 0)
 		(unit 1)
 		(exclude_from_sim no)
@@
 		(fields_autoplaced yes)
 		(property "Reference" "H3"
-			(at 165.1 102.8699 0)
+			(at 135.89 182.8799 0)
 			(effects
 				(font
@@
 		)
 		(property "Value" "MountingHole"
-			(at 165.1 105.4099 0)
+			(at 135.89 185.4199 0)
 			(effects
 				(font
@@
 		)
 		(property "Footprint" "MountingHole:MountingHole_3.2mm_M3"
-			(at 162.56 104.14 0)
+			(at 133.35 184.15 0)
 			(effects
 				(font
@@
 		)
 		(property "Datasheet" "~"
-			(at 162.56 104.14 0)
+			(at 133.35 184.15 0)
 			(effects
 				(font
@@
 		)
 		(property "Description" "Mounting Hole without connection"
-			(at 162.56 104.14 0)
+			(at 133.35 184.15 0)
 			(effects
 				(font
@@
 					(unit 1)
 				)
+			)
+		)
+	)
+	(symbol
+		(lib_id "RF_Module:Ai-Thinker-Ra-02")
+		(at 54.61 160.02 0)
+		(unit 1)
+		(exclude_from_sim no)
+		(in_bom yes)
+		(on_board yes)
+		(dnp no)
+		(fields_autoplaced yes)
+		(property "Reference" "U3"
+			(at 56.8041 142.24 0)
+			(effects
+				(font
+					(size 1.27 1.27)
+				)
+				(justify left)
+			)
+		)
+		(property "Value" "Ai-Thinker-Ra-02"
+			(at 56.8041 144.78 0)
+			(effects
+				(font
+					(size 1.27 1.27)
+				)
+				(justify left)
+			)
+		)
+		(property "Footprint" "RF_Module:Ai-Thinker-Ra-01-LoRa"
+			(at 80.01 170.18 0)
+			(effects
+				(font
+					(size 1.27 1.27)
+				)
+				(hide yes)
+			)
+		)
+		(property "Datasheet" "http://wiki.ai-thinker.com/_media/lora/docs/c048ps01a1_ra-02_product_specification_v1.1.pdf"
+			(at 57.15 140.97 0)
+			(effects
+				(font
+					(size 1.27 1.27)
+				)
+				(hide yes)
+			)
+		)
+		(property "Description" "Ai-Thinker Ra-02 410-525 MHz LoRa Module, SPI interface, U.FL antenna connector"
+			(at 54.61 160.02 0)
+			(effects
+				(font
+					(size 1.27 1.27)
+				)
+				(hide yes)
+			)
+		)
+		(pin "6"
+		)
+		(pin "4"
+		)
+		(pin "7"
+		)
+		(pin "8"
+		)
+		(pin "9"
+		)
+		(pin "15"
+		)
+		(pin "14"
+		)
+		(pin "16"
+		)
+		(pin "5"
+		)
+		(pin "1"
+		)
+		(pin "11"
+		)
+		(pin "13"
+		)
+		(pin "10"
+		)
+		(pin "3"
+		)
+		(pin "12"
+		)
+		(pin "2"
+		)
+		(instances
+			(project "OBCv1"
+				(path "/135eabb8-3fb8-4685-8bb7-68467cc8933b"
+					(reference "U3")
+					(unit 1)
+				)

Commit message: updates
Connections:
- net GND: now reaches J2.A1 (GND), J2.A12 (GND), J2.B1 (GND), J2.B12 (GND)
- net GND: now also J2.S1 (SHIELD), U2.29 (GND), U2.3 (GND)
- net at J2.A4 (VBUS), J2.A9 (VBUS), J2.B4 (VBUS)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: now also U2.8 (VBUS)
- net at J2.A6 (D+): now also J2.B6 (D+), U2.4 (D+)
- net at J2.A7 (D-): now also J2.B7 (D-), U2.5 (D-)
Other:
- company: (none) -> AfriOrbit EduSpace
- title: (none) -> EduSat OBC & Communications Board
- moved on the sheet: J2, U2

Commit message: a
Parts:
- added C1: 100n, Capacitor_SMD:C_0805_2012Metric, symbol Device:C
- added D1, D2, D3: D_TVS, Diode_SMD:D_0603_1608Metric, symbol Device:D_TVS
- added R1, R2: 5k1, Resistor_SMD:R_0805_2012Metric, symbol Device:R
- added R3: 22.1k, symbol Device:R
- added R4: 47.5k, symbol Device:R
Connections:
- net GND: now also C1.2, D1.1 (A1), D2.1 (A1), D3.1 (A1), R1.1, R2.1, R4.2
- net +5V_VBUS: now reaches J2.A4 (VBUS), J2.A9 (VBUS), J2.B4 (VBUS), J2.B9 (VBUS)
- net +5V_VBUS: now also C1.1, D1.2 (A2), R3.1; no longer U2.8 (VBUS)
- net at J2.A5 (CC1): now also R1.2
- net at J2.A6 (D+), J2.B6 (D+), U2.4 (D+): now also D3.2 (A2)
- net at J2.A7 (D-), J2.B7 (D-), U2.5 (D-): now also D2.2 (A2)
- net at J2.B5 (CC2): now also R2.2
- new net: R3.2, R4.1, U2.8 (VBUS)
Other:
- moved on the sheet: J1, J2, U2

Commit message: Updates
Parts:
- added C2, C3: 100n, Capacitor_SMD:C_0805_2012Metric, symbol Device:C
- added C4: 4.7u, Capacitor_SMD:C_0805_2012Metric, symbol Device:C
- added Q1, Q2: MMBT9014C, Package_TO_SOT_SMD:SOT-23, symbol Transistor_BJT:BC848
- added R5: 1k, symbol Device:R
- added R6, R7: 10k, symbol Device:R
- added S1: RESET, PTS647SM50SMTR2LFS, symbol PTS647SM50SMTR2LFS:PTS647SM50SMTR2LFS
- added S2: BOOT, PTS647SM50SMTR2LFS, symbol PTS647SM50SMTR2LFS:PTS647SM50SMTR2LFS
Connections:
- net GND: now also MICRO_SD1.6 (VSS), MICRO_SD1.MP1 (SHIELD), MICRO_SD1.MP2 (SHIELD), MICRO_SD1.MP3 (SHIELD), MICRO_SD1.MP4 (SHIELD), U1.1 (GND), U1.15 (GND), U1.38 (GND), U1.39 (GND), U3.1 (GND), U3.16 (GND), U3.2 (GND), U3.9 (GND), C2.2, C3.2, C4.2
- net CS_SD: now reaches MICRO_SD1.2 (CD/DAT3)
- net MOSI: now reaches MICRO_SD1.3 (CMD)
- net MOSI: now also J1.20 (Pin_20), U3.14 (MOSI)
- net +3.3V: now reaches MICRO_SD1.4 (VDD)
- net +3.3V: now also J1.2 (Pin_2), U2.6 (VDD), U2.7 (VREGIN), U3.3 (VDD), C2.1, C3.1, C4.1, R5.1
- net SCK: now reaches MICRO_SD1.5 (CLK)
- net SCK: now also J1.24 (Pin_24), U3.12 (SCK)
- net MISO: now reaches MICRO_SD1.7 (DAT0)
- net MISO: now also J1.22 (Pin_22), U3.13 (MISO)
- net +5V: now reaches J1.1 (Pin_1)
- net SDA: now reaches J1.4 (Pin_4)
- net SCL: now reaches J1.6 (Pin_6)
- net TXD: now reaches J1.7 (Pin_7)
- net RXD: now reaches J1.9 (Pin_9)
- net RTS: now reaches U2.24 (~{RTS})
- net RTS: now also Q1.2 (E), R7.1
- net at U2.25 (RXD): now also U1.35 (TXD0/IO1)
- net at U2.26 (TXD): now also U1.34 (RXD0/IO3)
- net DTR: now reaches U2.28 (~{DTR})
- net DTR: now also Q2.2 (E), R6.1
- net at U2.9 (~{RST}): now also R5.2
- net CS_LM: now reaches U3.15 (~{NSS})
- new net: Q2.1 (B), R7.2
- new net: Q1.1 (B), R6.2
- new net EN: Q1.3 (C), S1.1
- new net IO0_BTN: Q2.3 (C), S2.1
- no-connect marks 0 -> 28
Other:
- moved on the sheet: C1, D1, D2, D3, H1, H2, H3, H4, J1, J2, MICRO_SD1, R1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

Commit message: OBC updates
Parts:
- added C5, C6, C7, C8: 100n, Capacitor_SMD:C_0805_2012Metric, symbol Device:C
- added C9: 22u, Capacitor_SMD:C_0805_2012Metric, symbol Device:C
- added R8, R9: 10k, Resistor_SMD:R_0805_2012Metric_Pad1.20x1.40mm_HandSolder, symbol Device:R
- R3, R4, R5, R6, R7: footprint (none) -> Resistor_SMD:R_0805_2012Metric_Pad1.20x1.40mm_HandSolder
- S1, S2: footprint PTS647SM50SMTR2LFS -> KiCad:PTS647SM50SMTR2LFS
Connections:
- net +3.3V: now also U1.2 (VDD), C8.1, C9.1, R8.2, R9.2
- net CS_LM: now also U1.23 (IO15)
- net CS_SD: now also U1.24 (IO2)
- net EN: now also S1.2, U1.3 (EN), C5.1, C7.1, R8.1
- net GND: now also S1.3, S1.4, S2.3, S2.4, C5.2, C6.2, C7.2, C8.2, C9.2
- net IO0_BTN: now also S2.2, U1.25 (IO0), C6.1, R9.1
- net MISO: now also U1.30 (IO18)
- net MOSI: now also U1.31 (IO19)
- net RXD: now also U1.27 (IO16)
- net SCK: now also U1.37 (IO23)
- net SCL: now also U1.36 (IO22)
- net SDA: now also U1.33 (IO21)
- net TXD: now also U1.28 (IO17)
- net D1: now reaches U1.10 (IO25)
- net ANA2: now reaches U1.11 (IO26)
- net VSYNC: now reaches U1.12 (IO27)
- net PCLK: now reaches U1.13 (IO14)
- net D2: now reaches U1.14 (IO12)
- net D0: now reaches U1.16 (IO13)
- net DHT: now reaches U1.26 (IO4)
- net XCLK: now reaches U1.29 (IO5)
- net ANA1: now reaches U1.4 (SENSOR_VP)
- net ANA3: now reaches U1.5 (SENSOR_VN)
- net UV: now reaches U1.6 (IO34)
- net D7: now reaches U1.7 (IO35)
- net D5: now reaches U1.8 (IO32)
- net D3: now reaches U1.9 (IO33)

Commit message: Updates
Parts:
- added J3: IDC Connector 2x10 20P, Connector_IDC:IDC-Header_2x10_P2.54mm_Horizontal, symbol Connector:Conn_ARM_JTAG_SWD_20
- S1: value RESET -> RESET/EN
Connections:
- net +3.3V: now also J3.1 (VCC)
- net +5V: now also J1.38 (Pin_38); no longer J1.1 (Pin_1)
- net ANA1: now also J1.6 (Pin_6)
- net ANA2: now also J1.20 (Pin_20)
- net ANA3: now also J1.8 (Pin_8)
- net D0: now also J3.16 (D0)
- net D1: now also J3.15 (D1)
- net D2: now also J3.14 (D2)
- net D3: now also J3.13 (D3)
- net D5: now also J3.11 (D5)
- net D7: now also J3.9 (D7)
- net DHT: now also J1.25 (Pin_25)
- net EN: now also J1.4 (Pin_4)
- net GND: now also J1.1 (Pin_1), J1.13 (Pin_13), J1.28 (Pin_28), J3.2 (GND)
- net MISO: now also J1.15 (Pin_15), J3.12 (D4); no longer J1.22 (Pin_22)
- net MOSI: now also J1.3 (Pin_3), J3.10 (D6); no longer J1.20 (Pin_20)
- net PCLK: now also J3.7 (PCLK)
- net RXD: now also J1.23 (Pin_23); no longer J1.9 (Pin_9)
- net SCK: now also J1.17 (Pin_17), J3.6 (HREF); no longer J1.24 (Pin_24)
- net SCL: now also J1.5 (Pin_5), J3.3 (SIOC); no longer J1.6 (Pin_6)
- net SDA: now also J1.11 (Pin_11), J3.4 (SIOD); no longer J1.4 (Pin_4)
- net TXD: now also J1.21 (Pin_21); no longer J1.7 (Pin_7)
- net UV: now also J1.10 (Pin_10)
- net VSYNC: now also J3.5 (VSYNC)
- net XCLK: now also J3.8 (XCLK)
- net +BATT: now reaches J1.39 (Pin_39)
- net +BATT: now also J1.40 (Pin_40)
- no-connect marks 28 -> 50
Other:
- note added: "Camera Connector"

Commit message: Uploads
Other:
- moved on the sheet: C5, C6, Q1, Q2, R6, R7, R9, S1, S2

Commit message: Routing
Connections:
- net D+: now reaches D3.2 (A2), J2.A6 (D+), J2.B6 (D+), U2.4 (D+)
- net D-: now reaches D2.2 (A2), J2.A7 (D-), J2.B7 (D-), U2.5 (D-)
Changed lines of the file:
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@@
+		)
+	)
+	(label "D-"
+		(at 173.99 45.72 0)
+		(fields_autoplaced yes)
+		(effects
+			(font
+				(size 1.27 1.27)
+			)
+			(justify left bottom)
 		)
 	)
@@
 		)
 	)
+	(label "D+"
+		(at 173.99 48.26 0)
+		(fields_autoplaced yes)
+		(effects
+			(font
+				(size 1.27 1.27)
+			)
+			(justify left bottom)
+		)
+	)
