File: EduSat v2/OBCv1/OBCv1.kicad_sch (KiCad schematic)
At the start: 36 parts, among them J1 Conn_02x20_Odd_Even, J2 USB_C_Receptacle_USB2.0_16P, J3 IDC Connector 2x10 20P, Q1 MMBT9014C, Q2 MMBT9014C, U1 ESP32-WROOM-32E, U2 CP2102N-Axx-xQFN28, U3 Ai-Thinker-Ra-02

Commit message: EPS and OBC done
Connections:
- net +5V: now also J1.1 (Pin_1)
- net GND: no longer J1.1 (Pin_1)
Changed lines of the file:
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@@
 	)
 	(junction
-		(at 135.89 139.7)
-		(diameter 0)
-		(color 0 0 0 0)
-	)
-	(junction
 		(at 238.76 48.26)
 		(diameter 0)
@@
 	(wire
 		(pts
+			(xy 133.35 124.46) (xy 152.4 124.46)
+		)
+		(stroke
+			(width 0)
+			(type default)
+		)
+	)
+	(wire
+		(pts
 			(xy 64.77 109.22) (xy 71.12 109.22)
 		)
@@
 	(wire
 		(pts
-			(xy 135.89 124.46) (xy 135.89 139.7)
-		)
-		(stroke
-			(width 0)
-			(type default)
-		)
-	)
-	(wire
-		(pts
 			(xy 195.58 133.35) (xy 203.2 133.35)
 		)
@@
 	(wire
 		(pts
-			(xy 133.35 124.46) (xy 135.89 124.46)
-		)
-		(stroke
-			(width 0)
-			(type default)
-		)
-	)
-	(wire
-		(pts
 			(xy 234.95 48.26) (xy 238.76 48.26)
 		)
@@
 					(unit 1)
 				)
+			)
+		)
+	)
+	(symbol
+		(lib_id "power:+5V")
+		(at 152.4 124.46 0)
+		(unit 1)
+		(exclude_from_sim no)
+		(in_bom yes)
+		(on_board yes)
+		(dnp no)
+		(property "Reference" "#PWR036"
+			(at 152.4 128.27 0)
+			(effects
+				(font
+					(size 1.27 1.27)
+				)
+				(hide yes)
+			)
+		)
+		(property "Value" "+5V"
+			(at 152.4 120.904 0)
+			(effects
+				(font
+					(size 1.27 1.27)
+				)
+			)
+		)
+		(property "Footprint" ""
+			(at 152.4 124.46 0)
+			(effects
+				(font
+					(size 1.27 1.27)
+				)
+				(hide yes)
+			)
+		)
+		(property "Datasheet" ""
+			(at 152.4 124.46 0)
+			(effects
+				(font
+					(size 1.27 1.27)
+				)
+				(hide yes)
+			)
+		)
+		(property "Description" "Power symbol creates a global label with name \"+5V\""
+			(at 152.4 124.46 0)
+			(effects
+				(font
+					(size 1.27 1.27)
+				)
+				(hide yes)
+			)
+		)
+		(pin "1"
+		)
+		(instances
+			(project "OBCv1"
+				(path "/135eabb8-3fb8-4685-8bb7-68467cc8933b"
+					(reference "#PWR036")
+					(unit 1)
+				)
