File: EduSat v2/OBCv1/OBCv1.kicad_pcb (KiCad board)
At the start: 2 copper layers, 80.5 x 80.5 mm, 9 parts, among them J1 Conn_02x20_Odd_Even, J2 USB_C_Receptacle_USB2.0_16P, U1 ESP32-WROOM-32E, U2 CP2102N-Axx-xQFN28

Commit message: Another upload
Parts:
- added U3: Ai-Thinker-Ra-02, RF_Module:Ai-Thinker-Ra-01-LoRa, F.Cu at (59.8, 75.0)

Commit message: More updates
Parts:
- moved J1 0.18 mm to (67.0, 49.9)
Changed lines of the file:
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@@
 		(allow_soldermask_bridges_in_footprints no)
 		(aux_axis_origin 50.8 127)
-		(grid_origin 50.8 127)
+		(grid_origin 91.070259 86.735491)
 		(pcbplotparams
 			(layerselection 0x00010fc_ffffffff)
@@
 		(tags "USB C Type-C Receptacle SMD")
 		(property "Reference" "J2"
-			(at 0 -5.715 270)
+			(at 0 -5.715 -90)
 			(layer "F.SilkS")
 			(effects
@@
 		)
 		(fp_text user "${REFERENCE}"
-			(at 0 0 270)
+			(at 0 0 -90)
 			(layer "F.Fab")
 			(effects
@@
 		(locked yes)
 		(layer "F.Cu")
-		(at 66.940388 49.710258 90)
+		(at 66.970259 49.885491 90)
 		(descr "Through hole straight socket strip, 2x20, 2.54mm pitch, double cols (from Kicad 4.0.7), script generated")
 		(tags "Through hole socket strip THT 2x20 2.54mm double row")
 		(property "Reference" "J1"
-			(at -1.27 -2.77 270)
+			(at -1.27 -2.77 -90)
 			(layer "F.SilkS")
 			(effects
@@
 		)
 		(fp_text user "${REFERENCE}"
-			(at -1.27 24.13 360)
+			(at -1.27 24.13 0)
 			(layer "F.Fab")
 			(effects
@@
 		(tags "LoRa Ra-01")
 		(property "Reference" "U3"
-			(at 0 -1 270)
+			(at 0 -1 -90)
 			(layer "F.SilkS")
 			(effects
@@
 		)
 		(property "Value" "Ai-Thinker-Ra-02"
-			(at 0 9.75 270)
+			(at 0 9.75 -90)
 			(layer "F.Fab")
 			(effects
@@
 		)
 		(fp_text user "${REFERENCE}"
-			(at 0 1 270)
+			(at 0 1 -90)
 			(layer "F.Fab")
 			(effects
@@
 			)
 			(layer "F.Fab")
-			(net 7471205)
 		)
 		(fp_line
@@
 			)
 			(layer "F.Fab")
-			(net 7471205)
 		)
 		(fp_line
@@
 			)
 			(layer "F.Fab")
-			(net 7471205)
 		)
 		(fp_line
@@
 			)
 			(layer "F.Fab")
-			(net 7471205)
 		)
 		(fp_line
@@
 			)
 			(layer "F.Fab")
-			(net 7471205)
 		)
 		(fp_line
@@
 			)
 			(layer "F.Fab")
-			(net 7471205)
 		)
 		(fp_line
@@
 			)
 			(layer "F.Fab")
-			(net 7471205)
 		)
 		(fp_line
@@
 			)
 			(layer "F.Fab")
-			(net 7471205)
 		)
 		(fp_line
@@
 			)
 			(layer "F.Fab")
-			(net 7471205)
 		)
 		(fp_line
@@
 			)
 			(layer "F.Fab")
-			(net 7471205)
 		)
 		(fp_line
@@
 			)
 			(layer "F.Fab")
-			(net 7471205)
 		)
 		(fp_line
@@
 			)
 			(layer "F.Fab")
-			(net 7471205)
 		)
 		(fp_line
@@
 			)
 			(layer "F.Fab")
-			(net 7471205)
 		)
 		(fp_line
@@
 			)
 			(layer "F.Fab")
-			(net 7471205)
 		)
 		(fp_line
@@
 			)
 			(layer "F.Fab")
-			(net 7471205)
 		)
 		(fp_text user "Antenna"
@@
 		(start 50.801388 49.710258)
 		(end 50.8 123.75)
+		(locked yes)
 		(stroke
 			(width 0.1)
@@
 		(mid 51.751903 126.048097)
 		(end 50.8 123.75)
+		(locked yes)
 		(stroke
 			(width 0.1)
@@
 		(mid 51.753291 47.412161)
 		(end 54.051388 46.460258)
+		(locked yes)
 		(stroke
 			(width 0.1)
@@
 		(start 131.339824 49.732)
 		(end 131.339824 123.749705)
+		(locked yes)
 		(stroke
 			(width 0.1)
@@
 		(mid 130.387921 126.047802)
 		(end 128.089824 126.999705)
+		(locked yes)
 		(stroke
 			(width 0.1)
@@
 		(start 128.089824 126.999705)
 		(end 54.05 127)
+		(locked yes)
 		(stroke
 			(width 0.1)
@@
 		(start 54.051388 46.460258)
 		(end 128.089824 46.482)
+		(locked yes)
 		(stroke
 			(width 0.1)
@@
 		(mid 130.387921 47.433903)
 		(end 131.339824 49.732)
+		(locked yes)
 		(stroke
 			(width 0.1)

Commit message: OBC updates
Parts:
- added C1: 100n, Capacitor_SMD:C_0805_2012Metric, F.Cu at (141.7, 60.8)
- added C2: 100n, Capacitor_SMD:C_0805_2012Metric, F.Cu at (141.7, 63.8)
- added C3: 100n, Capacitor_SMD:C_0805_2012Metric, F.Cu at (141.7, 66.8)
- added C4: 4.7u, Capacitor_SMD:C_0805_2012Metric, F.Cu at (146.2, 60.8)
- added C5: 100n, Capacitor_SMD:C_0805_2012Metric, F.Cu at (146.2, 63.8)
- added C6: 100n, Capacitor_SMD:C_0805_2012Metric, F.Cu at (146.2, 66.8)
- added C7: 100n, Capacitor_SMD:C_0805_2012Metric, F.Cu at (150.6, 60.8)
- added C8: 100n, Capacitor_SMD:C_0805_2012Metric, F.Cu at (150.6, 63.8)
- added C9: 22u, Capacitor_SMD:C_0805_2012Metric, F.Cu at (150.6, 66.8)
- added D1: D_TVS, Diode_SMD:D_0603_1608Metric, F.Cu at (146.4, 69.6)
- added D2: D_TVS, Diode_SMD:D_0603_1608Metric, F.Cu at (146.4, 72.2)
- added D3: D_TVS, Diode_SMD:D_0603_1608Metric, F.Cu at (146.4, 74.8)
- added Q1: MMBT9014C, Package_TO_SOT_SMD:SOT-23, F.Cu at (142.0, 70.7)
- added Q2: MMBT9014C, Package_TO_SOT_SMD:SOT-23, F.Cu at (142.0, 75.3)
- added R1: 5k1, Resistor_SMD:R_0805_2012Metric, F.Cu at (150.7, 69.8)
- added R2: 5k1, Resistor_SMD:R_0805_2012Metric, F.Cu at (150.7, 72.7)
- added R3: 22.1k, Resistor_SMD:R_0805_2012Metric_Pad1.20x1.40mm_HandSolder, F.Cu at (141.1, 84.2)
- added R4: 47.5k, Resistor_SMD:R_0805_2012Metric_Pad1.20x1.40mm_HandSolder, F.Cu at (141.1, 87.2)
- added R5: 1k, Resistor_SMD:R_0805_2012Metric_Pad1.20x1.40mm_HandSolder, F.Cu at (141.1, 90.1)
- added R6: 10k, Resistor_SMD:R_0805_2012Metric_Pad1.20x1.40mm_HandSolder, F.Cu at (141.1, 93.1)
- added R7: 10k, Resistor_SMD:R_0805_2012Metric_Pad1.20x1.40mm_HandSolder, F.Cu at (141.1, 96.0)
- added R8: 10k, Resistor_SMD:R_0805_2012Metric_Pad1.20x1.40mm_HandSolder, F.Cu at (141.1, 99.0)
- added R9: 10k, Resistor_SMD:R_0805_2012Metric_Pad1.20x1.40mm_HandSolder, F.Cu at (141.1, 101.9)
- added S1: RESET, KiCad:PTS647SM50SMTR2LFS, F.Cu at (148.4, 86.5)
- added S2: BOOT, KiCad:PTS647SM50SMTR2LFS, F.Cu at (148.4, 94.1)
- moved J2 73.7 mm to (54.5, 62.3), turned to -90 degrees
- moved U3 51.3 mm to (111.1, 72.7), turned to 180 degrees
- moved U2 39.1 mm to (68.6, 72.7), turned to 90 degrees
- moved U1 28.8 mm to (66.7, 94.8), turned to 90 degrees
- moved MICRO_SD1 16.8 mm to (71.6, 118.7), turned to 0 degrees
Connections:
- net Net-(J2-VBUS-PadA4) renamed +5V_VBUS
- J1 pad 1: unconnected-(J1-Pin_1-Pad1) -> +5V
- J1 pad 2: unconnected-(J1-Pin_2-Pad2) -> +3.3V
- J1 pad 20: unconnected-(J1-Pin_20-Pad20) -> /MOSI
- J1 pad 22: unconnected-(J1-Pin_22-Pad22) -> /MISO
- J1 pad 24: unconnected-(J1-Pin_24-Pad24) -> /SCK
- J1 pad 4: unconnected-(J1-Pin_4-Pad4) -> /SDA
- J1 pad 6: unconnected-(J1-Pin_6-Pad6) -> /SCL
- J1 pad 7: unconnected-(J1-Pin_7-Pad7) -> /TXD
- J1 pad 9: unconnected-(J1-Pin_9-Pad9) -> /RXD
- J2 pad A1: Net-(J2-GND-PadA1) -> GND
- J2 pad A12: Net-(J2-GND-PadA1) -> GND
- J2 pad A5: unconnected-(J2-CC1-PadA5) -> Net-(J2-CC1)
- J2 pad A6: unconnected-(J2-D+-PadA6) -> Net-(D3-A2)
- J2 pad A7: unconnected-(J2-D--PadA7) -> Net-(D2-A2)
- J2 pad B1: Net-(J2-GND-PadA1) -> GND
- J2 pad B12: Net-(J2-GND-PadA1) -> GND
- J2 pad B5: unconnected-(J2-CC2-PadB5) -> Net-(J2-CC2)
- J2 pad B6: unconnected-(J2-D+-PadB6) -> Net-(D3-A2)
- J2 pad B7: unconnected-(J2-D--PadB7) -> Net-(D2-A2)
- J2 pad S1: unconnected-(J2-SHIELD-PadS1) -> GND
- MICRO_SD1 pad 2: unconnected-(MICRO_SD1-CD/DAT3-Pad2) -> /CS_SD
- MICRO_SD1 pad 3: unconnected-(MICRO_SD1-CMD-Pad3) -> /MOSI
- MICRO_SD1 pad 4: unconnected-(MICRO_SD1-VDD-Pad4) -> +3.3V
- MICRO_SD1 pad 5: unconnected-(MICRO_SD1-CLK-Pad5) -> /SCK
- MICRO_SD1 pad 6: unconnected-(MICRO_SD1-VSS-Pad6) -> GND
- MICRO_SD1 pad 7: unconnected-(MICRO_SD1-DAT0-Pad7) -> /MISO
- MICRO_SD1 pad MP1: unconnected-(MICRO_SD1-SHIELD-PadMP1) -> GND
- MICRO_SD1 pad MP2: unconnected-(MICRO_SD1-SHIELD-PadMP2) -> GND
- MICRO_SD1 pad MP3: unconnected-(MICRO_SD1-SHIELD-PadMP3) -> GND
- MICRO_SD1 pad MP4: unconnected-(MICRO_SD1-SHIELD-PadMP4) -> GND
- U1 pad 1: Net-(U1-GND-Pad1) -> GND
- U1 pad 10: unconnected-(U1-IO25-Pad10) -> /D1
- U1 pad 11: unconnected-(U1-IO26-Pad11) -> /ANA2
- U1 pad 12: unconnected-(U1-IO27-Pad12) -> /VSYNC
- U1 pad 13: unconnected-(U1-IO14-Pad13) -> /PCLK
- U1 pad 14: unconnected-(U1-IO12-Pad14) -> /D2
- U1 pad 15: Net-(U1-GND-Pad1) -> GND
- U1 pad 16: unconnected-(U1-IO13-Pad16) -> /D0
- U1 pad 2: unconnected-(U1-VDD-Pad2) -> +3.3V
- U1 pad 23: unconnected-(U1-IO15-Pad23) -> /CS_LM
- U1 pad 24: unconnected-(U1-IO2-Pad24) -> /CS_SD
- U1 pad 25: unconnected-(U1-IO0-Pad25) -> /IO0_BTN
- U1 pad 26: unconnected-(U1-IO4-Pad26) -> /DHT
- U1 pad 27: unconnected-(U1-IO16-Pad27) -> /RXD
- U1 pad 28: unconnected-(U1-IO17-Pad28) -> /TXD
- U1 pad 29: unconnected-(U1-IO5-Pad29) -> /XCLK
- U1 pad 3: unconnected-(U1-EN-Pad3) -> /EN
- U1 pad 30: unconnected-(U1-IO18-Pad30) -> /MISO
- U1 pad 31: unconnected-(U1-IO19-Pad31) -> /MOSI
- U1 pad 33: unconnected-(U1-IO21-Pad33) -> /SDA
- U1 pad 34: unconnected-(U1-RXD0/IO3-Pad34) -> Net-(U1-RXD0/IO3)
- U1 pad 35: unconnected-(U1-TXD0/IO1-Pad35) -> Net-(U1-TXD0/IO1)
- U1 pad 36: unconnected-(U1-IO22-Pad36) -> /SCL
- U1 pad 37: unconnected-(U1-IO23-Pad37) -> /SCK
- U1 pad 38: Net-(U1-GND-Pad1) -> GND
- U1 pad 39: Net-(U1-GND-Pad1) -> GND
- U1 pad 4: unconnected-(U1-SENSOR_VP-Pad4) -> /ANA1
- U1 pad 5: unconnected-(U1-SENSOR_VN-Pad5) -> /ANA3
- U1 pad 6: unconnected-(U1-IO34-Pad6) -> /UV
- U1 pad 7: unconnected-(U1-IO35-Pad7) -> /D7
- U1 pad 8: unconnected-(U1-IO32-Pad8) -> /D5
- U1 pad 9: unconnected-(U1-IO33-Pad9) -> /D3
- U2 pad 24: unconnected-(U2-~{RTS}-Pad24) -> /RTS
- U2 pad 25: unconnected-(U2-RXD-Pad25) -> Net-(U1-TXD0/IO1)
- U2 pad 26: unconnected-(U2-TXD-Pad26) -> Net-(U1-RXD0/IO3)
- U2 pad 28: unconnected-(U2-~{DTR}-Pad28) -> /DTR
- U2 pad 29: Net-(U2-GND-Pad29) -> GND
- U2 pad 3: Net-(U2-GND-Pad29) -> GND
- U2 pad 4: unconnected-(U2-D+-Pad4) -> Net-(D3-A2)
- U2 pad 5: unconnected-(U2-D--Pad5) -> Net-(D2-A2)
- U2 pad 6: unconnected-(U2-VDD-Pad6) -> +3.3V
- U2 pad 7: unconnected-(U2-VREGIN-Pad7) -> +3.3V
- U2 pad 8: unconnected-(U2-VBUS-Pad8) -> Net-(U2-VBUS)
- U2 pad 9: unconnected-(U2-~{RST}-Pad9) -> Net-(U2-~{RST})
- U3 pad 1: Net-(U3-GND-Pad1) -> GND
- U3 pad 12: unconnected-(U3-SCK-Pad12) -> /SCK
- U3 pad 13: unconnected-(U3-MISO-Pad13) -> /MISO
- U3 pad 14: unconnected-(U3-MOSI-Pad14) -> /MOSI
- U3 pad 15: unconnected-(U3-~{NSS}-Pad15) -> /CS_LM
- U3 pad 16: Net-(U3-GND-Pad1) -> GND
- U3 pad 2: Net-(U3-GND-Pad1) -> GND
- U3 pad 3: unconnected-(U3-VDD-Pad3) -> +3.3V
- U3 pad 9: Net-(U3-GND-Pad1) -> GND

Commit message: Updates
Parts:
- added J3: IDC Connector 2x10 20P, Connector_IDC:IDC-Header_2x10_P2.54mm_Horizontal, F.Cu at (110.2, 113.2)
- moved C8 100.5 mm to (59.6, 106.2), turned to 180 degrees
- moved C9 100.0 mm to (59.6, 108.2), turned to 180 degrees
- moved C7 99.2 mm to (63.6, 108.2), turned to 180 degrees
- moved RESET/EN 92.5 mm to (63.6, 123.2), turned to 180 degrees
- moved BOOT 80.8 mm to (73.1, 123.2), turned to 180 degrees
- moved R8 77.9 mm to (63.6, 106.2), turned to 180 degrees
- moved MICRO_SD1 57.7 mm to (124.0, 94.7), turned to 90 degrees
- moved U3 11.9 mm to (122.1, 68.2), turned to -90 degrees
- moved U2 2.70 mm to (66.0, 73.1), turned to -90 degrees
- moved U1 0.58 mm to (67.1, 94.4)
- renumbered S2 to BOOT, S1 to RESET/EN
Routing:
- added copper zone on F.Cu, net +3.3V
Other:
- copper layers 2 -> 4

Commit message: Uploads
Parts:
- S1: renamed from RESET/EN; value RESET -> RESET/EN
- moved R1 87.0 mm to (64.2, 59.9), turned to 90 degrees
- moved R2 87.0 mm to (64.2, 63.4), turned to -90 degrees
- moved D2 86.4 mm to (61.0, 59.6), turned to -90 degrees
- moved D3 86.3 mm to (61.0, 62.8), turned to 90 degrees
- moved D1 85.2 mm to (61.3, 66.3), turned to 180 degrees
- moved C1 84.4 mm to (57.7, 68.2), turned to 180 degrees
- moved R3 81.2 mm to (61.5, 68.2)
- moved C4 80.4 mm to (66.4, 70.6)
- moved R5 79.9 mm to (62.5, 76.2), turned to -90 degrees
- moved R4 78.0 mm to (65.5, 68.2)
- moved C3 75.6 mm to (66.4, 72.7)
- moved U2 4.61 mm to (67.0, 77.6)
- moved J2 1.10 mm to (54.5, 61.2)
- renumbered BOOT to S2
Connections:
- J1 pad 1: +5V -> GND
- J1 pad 10: unconnected-(J1-Pin_10-Pad10) -> /UV
- J1 pad 11: unconnected-(J1-Pin_11-Pad11) -> /SDA
- J1 pad 13: unconnected-(J1-Pin_13-Pad13) -> GND
- J1 pad 15: unconnected-(J1-Pin_15-Pad15) -> /MISO
- J1 pad 17: unconnected-(J1-Pin_17-Pad17) -> /SCK
- J1 pad 20: /MOSI -> /ANA2
- J1 pad 21: unconnected-(J1-Pin_21-Pad21) -> /TXD
- J1 pad 22: /MISO -> unconnected-(J1-Pin_22-Pad22)
- J1 pad 23: unconnected-(J1-Pin_23-Pad23) -> /RXD
- J1 pad 24: /SCK -> unconnected-(J1-Pin_24-Pad24)
- J1 pad 25: unconnected-(J1-Pin_25-Pad25) -> /DHT
- J1 pad 28: unconnected-(J1-Pin_28-Pad28) -> GND
- J1 pad 3: unconnected-(J1-Pin_3-Pad3) -> /MOSI
- J1 pad 38: unconnected-(J1-Pin_38-Pad38) -> +5V
- J1 pad 39: unconnected-(J1-Pin_39-Pad39) -> +BATT
- J1 pad 4: /SDA -> /EN
- J1 pad 40: unconnected-(J1-Pin_40-Pad40) -> +BATT
- J1 pad 5: unconnected-(J1-Pin_5-Pad5) -> /SCL
- J1 pad 6: /SCL -> /ANA1
- J1 pad 7: /TXD -> unconnected-(J1-Pin_7-Pad7)
- J1 pad 8: unconnected-(J1-Pin_8-Pad8) -> /ANA3
- J1 pad 9: /RXD -> unconnected-(J1-Pin_9-Pad9)
Routing:
- net /D7: track 0.00 -> 47.9 mm, vias 0 -> 1
- net /D5: track 0.00 -> 43.5 mm, vias 0 -> 1
- net /D3: track 0.00 -> 38.6 mm, vias 0 -> 1
- net /D1: track 0.00 -> 34.0 mm, vias 0 -> 1
- net /EN: track 0.00 -> 25.1 mm
- net Net-(U1-RXD0/IO3): track 0.00 -> 16.1 mm
- net Net-(U1-TXD0/IO1): track 0.00 -> 15.7 mm
- net Net-(U2-VBUS): track 0.00 -> 11.6 mm
- net Net-(J2-CC2): track 0.00 -> 6.92 mm
- net Net-(J2-CC1): track 0.00 -> 6.44 mm
- net Net-(D3-A2): track 0.00 -> 6.14 mm
- net Net-(D2-A2): track 0.00 -> 5.78 mm
- net Net-(U2-~{RST}): track 0.00 -> 2.30 mm
- added copper zone on F.Cu, net +5V_VBUS
- added copper zone on F.Cu, net Net-(U2-VBUS)

Commit message: Routing
Connections:
- net Net-(D2-A2) renamed /D-
- net Net-(D3-A2) renamed /D+
Routing:
- net /D+: track 6.14 -> 32.8 mm, vias 0 -> 2
- net /D-: track 5.78 -> 30.6 mm, vias 0 -> 2

Commit message: Routing
Parts:
- moved C5 94.8 mm to (63.6, 110.2), turned to 180 degrees
- moved C6 69.6 mm to (78.9, 84.5), turned to -90 degrees
- moved R6 68.8 mm to (74.4, 76.4), turned to -90 degrees
- moved R7 68.6 mm to (74.4, 80.2), turned to 90 degrees
- moved Q1 64.9 mm to (77.8, 80.4)
- moved Q2 64.2 mm to (77.8, 74.5)
- moved R9 62.6 mm to (81.0, 84.4), turned to -90 degrees
- moved MICRO_SD1 27.1 mm to (123.8, 67.6)
- moved U3 23.5 mm to (122.6, 91.7)
- moved C2 23.1 mm to (126.6, 81.2)
Routing:
- net /MOSI: track 0.00 -> 227.6 mm, vias 0 -> 3
- net /SCK: track 0.00 -> 187.7 mm, vias 0 -> 4
- net /MISO: track 0.00 -> 183.1 mm, vias 0 -> 3
- net /SDA: track 0.00 -> 143.4 mm, vias 0 -> 3
- net /SCL: track 0.00 -> 139.7 mm, vias 0 -> 4
- net /ANA2: track 0.00 -> 85.7 mm, vias 0 -> 2
- net /CS_LM: track 0.00 -> 65.3 mm
- net /ANA3: track 0.00 -> 64.9 mm, vias 0 -> 1
- net /ANA1: track 0.00 -> 63.1 mm, vias 0 -> 1
- net /UV: track 0.00 -> 62.1 mm, vias 0 -> 1
- net /CS_SD: track 0.00 -> 60.4 mm, vias 0 -> 2
- net /XCLK: track 0.00 -> 58.8 mm, vias 0 -> 2
- net /VSYNC: track 0.00 -> 51.1 mm, vias 0 -> 1
- net /DHT: track 0.00 -> 45.4 mm, vias 0 -> 1
- net /PCLK: track 0.00 -> 45.3 mm, vias 0 -> 1
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