File: EduSat v2/OBCv1/OBCv1.kicad_pcb (KiCad board)
At the start: 4 copper layers, 80.5 x 80.5 mm, 36 parts, among them J1 Conn_02x20_Odd_Even, J2 USB_C_Receptacle_USB2.0_16P, J3 IDC Connector 2x10 20P, Q1 MMBT9014C, Q2 MMBT9014C, U1 ESP32-WROOM-32E, U2 CP2102N-Axx-xQFN28, U3 Ai-Thinker-Ra-02

Commit message: UPDATES
Parts:
- renumbered S2 to BOOT, S1 to RESET/EN
Routing:
- net /EN: track 67.5 -> 111.5 mm, vias 1 -> 3
- net /IO0_BTN: track 21.1 -> 57.9 mm, vias 0 -> 4
- net +3.3V: track 0.00 -> 2.86 mm, vias 0 -> 9
- net /ANA3: track 64.9 -> 65.5 mm
- net GND: vias 0 -> 18
- added copper zone on B.Cu, net +3.3V
- added copper zone on F.Cu, net GND
- added copper zone on In1.Cu, net GND
- added copper zone on In2.Cu, net GND

Commit message: obc
Parts:
- added G***: LOGO, LOGO, F.Cu at (91.1, 86.7)
- added G***: LOGO, LOGO, B.Cu at (91.6, 86.1)
- renumbered MICRO_SD1 to MICRO_SD
Routing:
- net GND: vias 18 -> 402
Other:
- board text added: "+3V3"
- board text added: "+5V"
- board text added: "ANA1"
- board text added: "ANA2"
- board text added: "ANA3"
- board text added: "BATT"
- board text added: "CAMERA CONNECTOR"
- board text added: "DHT"
- board text added: "EN"
- board text added: "ESP32 MODULE"
- board text added: "EduSat OBC and Comms Board"
- board text added: "GND"
- board text added: "LORA COMM MODULE"
- board text added: "MISO"
- board text added: "MOSI"
- board text added: "RXD"
- board text added: "SCK"
- board text added: "SCL"
- board text added: "SDA"
- board text added: "TXD"
- board text added: "UV"

Commit message: EPS and OBC done
Parts:
- renumbered MICRO_SD to MICRO_SD1, RESET/EN to S1, BOOT to S2
Connections:
- J1 pad 1: GND -> +5V
Routing:
- net +5V: track 0.00 -> 49.5 mm
- net +BATT: track 0.00 -> 2.54 mm
- net /MOSI: track 227.6 -> 228.4 mm, vias 3 -> 4
- net GND: vias 402 -> 404
Changed lines of the file:
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@@
 			(layers "*.Cu" "*.Mask")
 			(remove_unused_layers no)
-			(net 1 "GND")
+			(net 9 "+5V")
 			(pinfunction "Pin_1")
 			(pintype "passive")
@@
 		(descr "PTS647SM50SMTR2LFS-2")
 		(tags "Switch")
-		(property "Reference" "RESET/EN"
+		(property "Reference" "S1"
 			(at 0 4.5 0)
 			(layer "F.SilkS")
@@
 		(at 123.795259 67.635491 90)
 		(descr "<b>TF-01A-6</b><br>")
-		(property "Reference" "MICRO_SD"
-			(at 8.9 -1.725 180)
+		(property "Reference" "MICRO_SD1"
+			(at 8.9 -2.725 180)
 			(layer "F.SilkS")
 			(effects
@@
 		(descr "PTS647SM50SMTR2LFS-2")
 		(tags "Switch")
-		(property "Reference" "BOOT"
+		(property "Reference" "S2"
 			(at 0 4.5 0)
 			(layer "F.SilkS")
@@
 		)
 	)
-	(gr_text "GND"
+	(gr_text "+5V"
 		(at 72.870259 60.035491 90)
 		(layer "F.SilkS")
@@
 	)
 	(via
+		(at 113.970259 51.135491)
+		(size 0.6)
+		(drill 0.3)
+		(layers "F.Cu" "B.Cu")
+		(free yes)
+		(net 1)
+	)
+	(via
 		(at 84.070259 120.735491)
 		(size 0.6)
@@
 	)
 	(via
+		(at 69.570259 47.335491)
+		(size 0.6)
+		(drill 0.3)
+		(layers "F.Cu" "B.Cu")
+		(free yes)
+		(net 1)
+	)
+	(via
 		(at 130.070259 110.735491)
 		(size 0.6)
@@
 	)
 	(segment
+		(start 112.690259 51.755491)
+		(end 112.690259 52.425491)
+		(width 0.25)
+		(layer "F.Cu")
+		(net 9)
+	)
+	(segment
+		(start 68.670259 48.185491)
+		(end 110.770259 48.185491)
+		(width 0.5)
+		(layer "F.Cu")
+		(net 9)
+	)
+	(segment
+		(start 111.470259 48.885491)
+		(end 111.470259 50.535491)
+		(width 0.25)
+		(layer "F.Cu")
+		(net 9)
+	)
+	(segment
+		(start 110.770259 48.185491)
+		(end 111.470259 48.885491)
+		(width 0.25)
+		(layer "F.Cu")
+		(net 9)
+	)
+	(segment
+		(start 66.970259 49.885491)
+		(end 68.670259 48.185491)
+		(width 0.5)
+		(layer "F.Cu")
+		(net 9)
+	)
+	(segment
+		(start 111.470259 50.535491)
+		(end 112.690259 51.755491)
+		(width 0.25)
+		(layer "F.Cu")
+		(net 9)
+	)
+	(segment
 		(start 62.570259 87.935491)
 		(end 64.570259 87.935491)
@@
 	)
 	(segment
-		(start 125.570259 101.135491)
-		(end 124.070259 102.635491)
+		(start 122.770259 49.935491)
+		(end 122.770259 67.605691)
 		(width 0.2)
 		(layer "F.Cu")
@@
 	)
 	(segment
-		(start 125.570259 99.735491)
-		(end 125.570259 101.135491)
+		(start 125.570259 101.135491)
+		(end 124.070259 102.635491)
 		(width 0.2)
 		(layer "F.Cu")
@@
 	)
 	(segment
-		(start 111.870259 89.835491)
-		(end 111.870259 100.535491)
+		(start 125.570259 99.735491)
+		(end 125.570259 101.135491)
 		(width 0.2)
 		(layer "F.Cu")
@@
 	)
 	(segment
-		(start 122.840459 67.605691)
-		(end 122.540459 67.605691)
+		(start 70.770259 47.335491)
+		(end 70.970259 47.135491)
 		(width 0.2)
 		(layer "F.Cu")
@@
 	)
 	(segment
-		(start 122.770259 49.935491)
-		(end 122.770259 67.605691)
+		(start 111.870259 89.835491)
+		(end 111.870259 100.535491)
 		(width 0.2)
 		(layer "F.Cu")
@@
 	)
 	(segment
-		(start 72.260259 47.135491)
-		(end 119.970259 47.135491)
+		(start 122.840459 67.605691)
+		(end 122.540459 67.605691)
 		(width 0.2)
 		(layer "F.Cu")
@@
 	)
 	(segment
-		(start 69.510259 49.885491)
-		(end 72.260259 47.135491)
+		(start 125.570259 98.035491)
+		(end 125.570259 99.735491)
 		(width 0.2)
 		(layer "F.Cu")
@@
 	)
 	(segment
-		(start 125.570259 98.035491)
-		(end 125.570259 99.735491)
+		(start 122.770259 67.605691)
+		(end 122.540459 67.605691)
 		(width 0.2)
 		(layer "F.Cu")
@@
 	)
 	(segment
-		(start 122.770259 67.605691)
-		(end 122.540459 67.605691)
+		(start 70.970259 47.135491)
+		(end 119.970259 47.135491)
 		(width 0.2)
 		(layer "F.Cu")
@@
 	)
 	(via
+		(at 70.770259 47.335491)
+		(size 0.6)
+		(drill 0.3)
+		(layers "F.Cu" "B.Cu")
+		(net 18)
+	)
+	(via
 		(at 122.570259 102.635491)
 		(size 0.6)
@@
 	)
 	(segment
+		(start 69.510259 48.595491)
+		(end 69.510259 49.885491)
+		(width 0.2)
+		(layer "B.Cu")
+		(net 18)
+	)
+	(segment
 		(start 125.570259 70.335491)
 		(end 125.570259 98.035491)
@@
 	)
 	(segment
+		(start 70.770259 47.335491)
+		(end 69.510259 48.595491)
+		(width 0.2)
+		(layer "B.Cu")
+		(net 18)
+	)
+	(segment
 		(start 119.870259 119.435491)
 		(end 101.070259 119.435491)
@@
 		(net 51)
 	)
+	(segment
+		(start 115.230259 49.885491)
+		(end 115.230259 52.425491)
+		(width 0.5)
+		(layer "F.Cu")
+		(net 100)
+	)
 	(zone
 		(net 2)
@@
 	)
 	(zone
+		(net 0)
+		(net_name "")
+		(layer "F.Cu")
+		(hatch edge 0.5)
+		(connect_pads
+			(clearance 0)
+		)
+		(min_thickness 0.25)
+		(filled_areas_thickness no)
+		(keepout
+			(tracks not_allowed)
+			(vias not_allowed)
+			(pads not_allowed)
+			(copperpour not_allowed)
+			(footprints allowed)
+		)
+		(fill
+			(thermal_gap 0.5)
+			(thermal_bridge_width 0.5)
+		)
+		(polygon
+			(pts
+				(xy 71.270259 47.435491) (xy 71.170259 47.535491) (xy 71.170259 47.635491) (xy 71.270259 47.735491)
+				(xy 110.770259 47.735491) (xy 110.770259 47.435491)
+			)
+		)
+	)
+	(zone
 		(net 51)
 		(net_name "Net-(U2-VBUS)")
@@
 		(layer "F.Cu")
 		(hatch edge 0.5)
+		(priority 15)
 		(connect_pads yes
-			(clearance 0.5)
+			(clearance 0.15)
 		)
 		(min_thickness 0.25)
@@
 		(filled_areas_thickness no)
 		(fill yes
-			(thermal_gap 0.5)
+			(thermal_gap 0.3)
 			(thermal_bridge_width 0.5)
 		)
