File: EduSat v2/EPSv3/EPSv3.kicad_pcb (KiCad board)
At the start: 2 copper layers, 1 part

Commit message: EPS updates
Parts:
- added BT2: 1042, Battery_Holder_1:BAT_1042, F.Cu at (218.1, 80.0)
- added C1: 0.1uF, Capacitor_SMD:C_0805_2012Metric_Pad1.18x1.45mm_HandSolder, F.Cu at (135.4, 32.9)
- added D1: Yellow LED, LED_SMD:LED_0805_2012Metric_Pad1.15x1.40mm_HandSolder, F.Cu at (112.8, 50.9)
- added R1: 100Ω, Resistor_SMD:R_0805_2012Metric_Pad1.20x1.40mm_HandSolder, F.Cu at (112.8, 53.8)
- added R2: 1kΩ, Resistor_SMD:R_0805_2012Metric_Pad1.20x1.40mm_HandSolder, F.Cu at (135.4, 35.9)
- added R3: 100Ω, Resistor_SMD:R_0805_2012Metric_Pad1.20x1.40mm_HandSolder, F.Cu at (135.4, 38.9)
- added U1: ~, DW06D:SOT-23-6_L2.9-W1.6-P0.95-LS2.8-BR, F.Cu at (151.7, 43.1)
- added U2: IRLML6344TRPBF, IRLML6344TRPBF:SOT95P240X112-3N, F.Cu at (149.0, 53.1)
- BT1: footprint BatteryHolderSingle:BAT_1042 -> Battery_Holder_1:BAT_1042
- moved BT1 19.3 mm to (218.2, 51.4)
Connections:
- BT1 pad N: unconnected-(BT1-PadN) -> Net-(U2-D)
- BT1 pad P: unconnected-(BT1-PadP) -> Net-(D1-K)

Commit message: EPS Schematics
Parts:
- added C1: 1n, Capacitor_SMD:C_0805_2012Metric_Pad1.18x1.45mm_HandSolder, F.Cu at (236.0, 119.3)
- added C10: 22u, Capacitor_SMD:C_0805_2012Metric_Pad1.18x1.45mm_HandSolder, F.Cu at (180.1, 118.1)
- added C11: 1n, Capacitor_SMD:C_0805_2012Metric_Pad1.18x1.45mm_HandSolder, F.Cu at (236.0, 125.3)
- added C12: 0.1u, Capacitor_SMD:C_0805_2012Metric_Pad1.18x1.45mm_HandSolder, F.Cu at (236.0, 122.3)
- added C2: 0.1u, Capacitor_SMD:C_0805_2012Metric_Pad1.18x1.45mm_HandSolder, F.Cu at (236.0, 116.3)
- added C3: 10u, Capacitor_SMD:C_0805_2012Metric_Pad1.18x1.45mm_HandSolder, F.Cu at (180.1, 100.1)
- added C4: 10u, Capacitor_SMD:C_0805_2012Metric_Pad1.18x1.45mm_HandSolder, F.Cu at (180.1, 106.1)
- added C6: 22u, Capacitor_SMD:C_0805_2012Metric_Pad1.18x1.45mm_HandSolder, F.Cu at (180.1, 103.1)
- added C7: 22u, Capacitor_SMD:C_0805_2012Metric_Pad1.18x1.45mm_HandSolder, F.Cu at (180.1, 109.1)
- added C8: 22u, Capacitor_SMD:C_0805_2012Metric_Pad1.18x1.45mm_HandSolder, F.Cu at (180.1, 112.1)
- added C9: 22u, Capacitor_SMD:C_0805_2012Metric_Pad1.18x1.45mm_HandSolder, F.Cu at (180.1, 115.1)
- added D1: DFLS130L-7, DFLS130L-7:DIO_DFLS130L-7, F.Cu at (79.5, 52.5)
- added D10: LED, LED_SMD:LED_0805_2012Metric_Pad1.15x1.40mm_HandSolder, F.Cu at (224.6, 132.9)
- added D2: DFLS130L-7, DFLS130L-7:DIO_DFLS130L-7, F.Cu at (79.5, 55.9)
- added D3: LED, LED_SMD:LED_0805_2012Metric_Pad1.15x1.40mm_HandSolder, F.Cu at (224.6, 126.8)
- added D4: LED, LED_SMD:LED_0805_2012Metric_Pad1.15x1.40mm_HandSolder, F.Cu at (224.6, 129.8)
- added D5: 25% Red, LED_SMD:LED_0805_2012Metric_Pad1.15x1.40mm_HandSolder, F.Cu at (185.0, 100.1)
- added D6: 50% Red, LED_SMD:LED_0805_2012Metric_Pad1.15x1.40mm_HandSolder, F.Cu at (185.0, 103.1)
- added D7: 75% Red, LED_SMD:LED_0805_2012Metric_Pad1.15x1.40mm_HandSolder, F.Cu at (185.0, 106.2)
- added D8: 100% Green, LED_SMD:LED_0805_2012Metric_Pad1.15x1.40mm_HandSolder, F.Cu at (185.0, 109.2)
- added IC1: DW06D, DW06D:DW06D_SFE, F.Cu at (152.4, 41.1)
- added J1: Solar_Panel_1, Connector_JST:JST_XH_S2B-XH-A_1x02_P2.50mm_Horizontal, F.Cu at (50.6, 46.8)
- added J2: Solar_Panel_2, Connector_JST:JST_XH_S2B-XH-A_1x02_P2.50mm_Horizontal, F.Cu at (62.8, 46.8)
- added J3: USBPwrIn, Connector_USB:USB_C_Receptacle_GCT_USB4125-xx-x_6P_TopMnt_Horizontal, F.Cu at (234.7, 110.4)
- added J4: Release Detection, Connector_JST:JST_XH_S2B-XH-A_1x02_P2.50mm_Horizontal, F.Cu at (216.2, 128.6)
- added L1: 1uH, MCS0630-100MN1:INDPM7366X300N, F.Cu at (117.4, 72.9)
- added R1: 1k5, Resistor_SMD:R_0805_2012Metric_Pad1.20x1.40mm_HandSolder, F.Cu at (231.2, 116.3)
- added R10: 10k, Resistor_SMD:R_0805_2012Metric_Pad1.20x1.40mm_HandSolder, F.Cu at (184.9, 115.2)
- added R13: 1k5, Resistor_SMD:R_0805_2012Metric_Pad1.20x1.40mm_HandSolder, F.Cu at (231.2, 134.0)
- added R2: 7k5, Resistor_SMD:R_0805_2012Metric_Pad1.20x1.40mm_HandSolder, F.Cu at (231.2, 119.2)
- added R3: 30k, Resistor_SMD:R_0805_2012Metric_Pad1.20x1.40mm_HandSolder, F.Cu at (231.2, 122.2)
- added R4: 1k5, Resistor_SMD:R_0805_2012Metric_Pad1.20x1.40mm_HandSolder, F.Cu at (231.2, 131.0)
- added R5: 5k1, Resistor_SMD:R_0805_2012Metric_Pad1.20x1.40mm_HandSolder, F.Cu at (231.2, 125.1)
- added R6: 5k1, Resistor_SMD:R_0805_2012Metric_Pad1.20x1.40mm_HandSolder, F.Cu at (231.2, 128.1)
- added R7: 2R, Resistor_SMD:R_0805_2012Metric_Pad1.20x1.40mm_HandSolder, F.Cu at (184.9, 112.2)
- added R8: 0R5, Resistor_SMD:R_0805_2012Metric_Pad1.20x1.40mm_HandSolder, F.Cu at (184.9, 118.1)
- added S1: USB-Solar Toggle, SPDT Switch:SS12D10L3, F.Cu at (216.1, 110.4)
- added S2: Push-Button, Push_Button:PTS647SM50SMTR2LFS, F.Cu at (142.2, 76.1)
- added S3: Power Switch, SPDT Switch:SS12D10L3, F.Cu at (216.1, 120.3)
- added U2: IP5306, IP5306:SOIC9P127_490X600X170L84X42T330X241N, F.Cu at (112.9, 81.7)
- added U4: ACS712xLCTR-05B, Package_SO:SOIC-8_3.9x4.9mm_P1.27mm, F.Cu at (237.8, 130.2)
- U1: value ~ -> ACS712xLCTR-05B; footprint DW06D:SOT-23-6_L2.9-W1.6-P0.95-LS2.8-BR -> Package_SO:SOIC-8_3.9x4.9mm_P1.27mm
- moved U1 60.6 mm to (91.2, 45.2)
- renumbered BT2 to BT1, BT1 to BT2, C1 to C5, D1 to D9, R2 to R11, R1 to R12, R3 to R9, U2 to U3
Connections:
- BT1 pad P: Net-(D1-K) -> Net-(D9-K)
- BT2 pad P: Net-(D1-K) -> Net-(D9-K)
- C5 pad 1: Net-(D1-K) -> Net-(D9-K)
- C5 pad 2: Net-(U1-VDD) -> Net-(IC1-VDD)
- D9 pad 1: Net-(D1-K) -> Net-(D9-K)
- R11 pad 1: Net-(U1-V-) -> Net-(IC1-V-)
- R9 pad 1: Net-(D1-K) -> Net-(D9-K)
- U1 pad 1: Net-(U1-V-) -> Net-(D1-PadC)
- U1 pad 2: GND -> Net-(D1-PadC)
- U1 pad 3: Net-(D1-K) -> Net-(S1-NC)
- U1 pad 4: unconnected-(U1-D-Pad4) -> Net-(S1-NC)
- U1 pad 5: Net-(U1-VDD) -> GND
- U1 pad 6: Net-(D1-K) -> Net-(U1-FILTER)
- U3 pad 1: Net-(D1-K) -> Net-(D9-K)
- U3 pad 2: Net-(D1-K) -> Net-(D9-K)

Commit message: More updates
Parts:
- added H1: MountingHole, MountingHole:MountingHole_3.2mm_M3, F.Cu at (53.4, 123.0)
- added H2: MountingHole, MountingHole:MountingHole_3.2mm_M3, F.Cu at (127.4, 123.0)
- added H3: MountingHole, MountingHole:MountingHole_3.2mm_M3, F.Cu at (53.4, 49.0)
- added H4: MountingHole, MountingHole:MountingHole_3.2mm_M3, F.Cu at (127.4, 49.0)
- added J5: Conn_02x20_Odd_Even, Connector_PinSocket_2.54mm:PinSocket_2x20_P2.54mm_Vertical, F.Cu at (66.3, 49.2)
- BT1, BT2: value 1042 -> 1043; footprint Battery_Holder_1:BAT_1042 -> 1043:BAT_1043; moved to B.Cu
- moved R13 187.2 mm to (62.9, 52.0), turned to 90 degrees
- moved D10 183.1 mm to (61.9, 48.9)
- moved J4 172.2 mm to (59.5, 57.1), turned to -90 degrees
- moved U4 170.4 mm to (71.1, 94.9)
- moved C12 163.0 mm to (75.9, 91.5), turned to 90 degrees
- moved C11 162.6 mm to (75.9, 96.6), turned to -90 degrees
- moved J3 161.9 mm to (73.3, 122.8)
- moved R6 160.3 mm to (71.3, 117.3), turned to 180 degrees
- moved R5 156.0 mm to (75.4, 117.3)
- moved S3 154.1 mm to (62.2, 113.7), turned to 180 degrees
- moved R4 150.6 mm to (81.0, 120.8), turned to 90 degrees
- moved D4 144.2 mm to (81.0, 116.7), turned to -90 degrees
- moved C1 139.1 mm to (97.2, 109.4), turned to 180 degrees
- moved C2 134.1 mm to (102.0, 110.1), turned to -90 degrees
- moved BT2 129.9 mm to (90.4, 74.6)
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Connections:
- BT1 pad P: Net-(D9-K) -> +BATT
- BT2 pad P: Net-(D9-K) -> +BATT
- C5 pad 1: Net-(D9-K) -> Net-(IC1-S2)
- C7 pad 1: Net-(D9-K) -> +BATT
- D9 pad 1: Net-(D9-K) -> +BATT
- IC1 pad 3: Net-(D9-K) -> Net-(IC1-S2)
- IC1 pad 6: Net-(D9-K) -> Net-(IC1-S2)
- J4 pad 1: Net-(J4-Pin_1) -> +5V
- J4 pad 2: +5V -> Net-(J4-Pin_2)
- L1 pad 2: Net-(D9-K) -> +BATT
- R8 pad 1: Net-(D9-K) -> +BATT
- R9 pad 1: Net-(D9-K) -> +BATT
- R9 pad 2: GND -> Net-(IC1-VDD)
- S3 pad 2: Net-(J4-Pin_1) -> Net-(J4-Pin_2)
- U2 pad 6: Net-(D9-K) -> +BATT
- U3 pad 1: Net-(D9-K) -> +BATT
- U3 pad 2: Net-(D9-K) -> Net-(IC1-S2)
Other:
- board outline added: 80.5 x 80.5 mm

Commit message: EPS routing
Parts:
- moved S1 9.48 mm to (89.6, 113.8), turned to -90 degrees
Routing:
- net Net-(J1-Pin_1): track 0.00 -> 3.92 mm
- net Net-(J2-Pin_1): track 0.00 -> 3.90 mm
- net Net-(D3-A): track 0.00 -> 2.76 mm
- net Net-(J3-CC2): track 0.00 -> 2.73 mm
- net Net-(J3-CC1): track 0.00 -> 2.73 mm
- net Net-(U1-FILTER): track 0.00 -> 2.62 mm
- net Net-(D4-A): track 0.00 -> 2.05 mm
- added copper zone on F.Cu, net /ANA2
- added copper zone on F.Cu, net Net-(D1-PadC)
- added copper zone on F.Cu, net Net-(S1-NC)
- added copper zone on F.Cu, net Net-(S1-NO)

Commit message: EPS routing done
Parts:
- moved S2 28.7 mm to (120.2, 88.1), turned to 0 degrees
- moved R10 24.7 mm to (113.7, 86.3)
- moved D5 21.6 mm to (119.8, 101.5), turned to 180 degrees
- moved D6 18.1 mm to (119.8, 98.7), turned to 0 degrees
- moved D7 14.7 mm to (119.8, 95.9), turned to 180 degrees
- moved D8 11.4 mm to (119.8, 93.2), turned to 0 degrees
- moved R13 2.81 mm to (60.3, 50.9)
- moved D10 2.81 mm to (59.3, 47.8)
- moved D9 0.13 mm to (94.7, 70.4)
Routing:
- net +5V: track 0.00 -> 88.6 mm, vias 0 -> 6
- net /ANA1: track 0.00 -> 85.4 mm, vias 0 -> 1
- net /ANA2: track 0.00 -> 61.3 mm
- net /ANA3: track 0.00 -> 44.2 mm, vias 0 -> 1
- net Net-(D5-K): track 0.00 -> 39.1 mm
- net Net-(D5-A): track 0.00 -> 35.9 mm
- net Net-(D7-A): track 0.00 -> 32.3 mm
- net Net-(U2-KEY): track 0.00 -> 21.5 mm
- net Net-(IC1-S2): track 0.00 -> 9.90 mm
- net Net-(IC1-VDD): track 0.00 -> 4.88 mm
- net Net-(D9-A): track 0.00 -> 4.43 mm
- net Net-(R10-Pad2): track 0.00 -> 2.88 mm
- net Net-(C6-Pad1): track 0.00 -> 2.47 mm
- net Net-(U4-FILTER): track 0.00 -> 2.43 mm
- net Net-(C3-Pad1): track 0.00 -> 2.12 mm
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- added copper zone on F.Cu, net +5V
- added copper zone on F.Cu, net +BATT
- added copper zone on F.Cu, net /VIN
- added copper zone on F.Cu, net /VOUT
- added copper zone on B.Cu, net GND
- added copper zone on F.Cu, net GND
- added copper zone on B.Cu, net Net-(J4-Pin_2)
- added copper zone on F.Cu, net Net-(S3-NC)
- added copper zone on F.Cu, net Net-(U2-SW)
- added copper zone on F.Cu, net Net-(U3-D)
Other:
- board text added: "100%"
- board text added: "25%"
- board text added: "50%"
- board text added: "75%"

Commit message: Updates
Parts:
- added C13: 10u, Capacitor_SMD:C_0805_2012Metric_Pad1.18x1.45mm_HandSolder, F.Cu at (69.0, 60.9)
- added C14: 100n, Capacitor_SMD:C_0805_2012Metric_Pad1.18x1.45mm_HandSolder, F.Cu at (74.9, 62.9)
- added C15: 22u, Capacitor_SMD:C_0805_2012Metric_Pad1.18x1.45mm_HandSolder, F.Cu at (74.9, 56.6)
- added C16: 22u, Capacitor_SMD:C_0805_2012Metric_Pad1.18x1.45mm_HandSolder, F.Cu at (72.6, 56.6)
- added L2: 4.7uH, MCS0630-100MN1:INDPM7366X300N, F.Cu at (79.7, 60.9)
- added U5: AP63203WU, Package_TO_SOT_SMD:TSOT-23-6, F.Cu at (72.0, 60.8)
Connections:
- J5 pad 1: unconnected-(J5-Pin_1-Pad1) -> +5V
- J5 pad 2: unconnected-(J5-Pin_2-Pad2) -> +3.3V
Routing:
- net /ANA3: track 44.2 -> 48.6 mm
- net +5V: track 88.6 -> 84.2 mm
- net Net-(U5-BST): track 0.00 -> 1.92 mm
- added copper zone on F.Cu, net +3.3V
- added copper zone on F.Cu, net Net-(U5-SW)

Commit message: Updates
Parts:
- S1, S3: footprint SPDT Switch:SS12D10L3 -> SS-12D10L3:SS12D10L3
- S2: footprint Push_Button:PTS647SM50SMTR2LFS -> PTS647SM50SMTR2LFS:PTS647SM50SMTR2LFS
Connections:
- J5 pad 34: unconnected-(J5-Pin_34-Pad34) -> /ANA3
- J5 pad 36: unconnected-(J5-Pin_36-Pad36) -> /ANA2
- J5 pad 38: unconnected-(J5-Pin_38-Pad38) -> /ANA1
- J5 pad 39: unconnected-(J5-Pin_39-Pad39) -> +BATT
- J5 pad 40: unconnected-(J5-Pin_40-Pad40) -> +BATT
Routing:
- net +BATT: track 0.00 -> 25.1 mm
- net /ANA2: track 61.3 -> 85.4 mm
- net /ANA3: track 48.6 -> 71.9 mm
- net /ANA1: track 85.4 -> 107.4 mm

Commit message: EPS and OBC done
Parts:
- added G***: LOGO, LOGO, F.Cu at (111.5, 59.8)
- added G***: LOGO, LOGO, B.Cu at (90.4, 87.1)
Connections:
- J5 pad 20: unconnected-(J5-Pin_20-Pad20) -> /ANA2
- J5 pad 34: /ANA3 -> unconnected-(J5-Pin_34-Pad34)
- J5 pad 36: /ANA2 -> unconnected-(J5-Pin_36-Pad36)
- J5 pad 38: /ANA1 -> +5V
- J5 pad 6: unconnected-(J5-Pin_6-Pad6) -> /ANA1
- J5 pad 8: unconnected-(J5-Pin_8-Pad8) -> /ANA3
Routing:
- net +5V: track 84.2 -> 135.6 mm
- net /ANA1: track 107.4 -> 148.1 mm
- net /ANA3: track 71.9 -> 54.5 mm
- net /ANA2: track 85.4 -> 102.6 mm
- net GND: vias 0 -> 337
Other:
- board text added: "EduSat EPS Board"
- board text added: "OFF"
- board text added: "ON"
