File: EduSat v2/EPSv3/EPSv3.kicad_sch (KiCad schematic)
At the start: 1 part

Commit message: EPS updates
Parts:
- removed BT1: 1042, BatteryHolderSingle:BAT_1042, symbol 1042:1042
- added BT1, BT2: 1042, Battery_Holder_1:BAT_1042, symbol Battery_Holder_1:1042
- added C1: 0.1uF, Capacitor_SMD:C_0805_2012Metric_Pad1.18x1.45mm_HandSolder, symbol Device:C
- added D1: Yellow LED, LED_SMD:LED_0805_2012Metric_Pad1.15x1.40mm_HandSolder, symbol Device:LED
- added R1, R3: 100Ω, Resistor_SMD:R_0805_2012Metric_Pad1.20x1.40mm_HandSolder, symbol Device:R
- added R2: 1kΩ, Resistor_SMD:R_0805_2012Metric_Pad1.20x1.40mm_HandSolder, symbol Device:R
- added U1: ~, DW06D:SOT-23-6_L2.9-W1.6-P0.95-LS2.8-BR, symbol DW06D:DW06D
- added U2: IRLML6344TRPBF, IRLML6344TRPBF:SOT95P240X112-3N, symbol IRLML6344TRPBF:IRLML6344TRPBF
Connections:
- new net: BT1.P, BT2.P, C1.1, D1.1 (K), R3.1, U1.3 (S2), U1.6 (VSS), U2.1 (G), U2.2 (S)
- new net: D1.2 (A), R1.1
- new net: BT1.N, BT2.N, R1.2, U2.3 (D)
- new net: R2.1, U1.1 (V-)
- new net: C1.2, U1.5 (VDD)
- new net GND: R2.2, R3.2, U1.2 (S1)

Commit message: EPS Schematics
Parts:
- removed U1: ~, DW06D:SOT-23-6_L2.9-W1.6-P0.95-LS2.8-BR, symbol DW06D:DW06D
- added C1, C11: 1n, Capacitor_SMD:C_0805_2012Metric_Pad1.18x1.45mm_HandSolder, symbol Device:C
- added C10, C6, C7, C8, C9: 22u, Capacitor_SMD:C_0805_2012Metric_Pad1.18x1.45mm_HandSolder, symbol Device:C
- added C12, C2: 0.1u, Capacitor_SMD:C_0805_2012Metric_Pad1.18x1.45mm_HandSolder, symbol Device:C
- added C3, C4: 10u, Capacitor_SMD:C_0805_2012Metric_Pad1.18x1.45mm_HandSolder, symbol Device:C
- added D1, D2: DFLS130L-7, DFLS130L-7:DIO_DFLS130L-7, symbol DFLS130L-7:DFLS130L-7
- added D10, D3, D4: LED, LED_SMD:LED_0805_2012Metric_Pad1.15x1.40mm_HandSolder, symbol Device:LED
- added D5: 25% Red, LED_SMD:LED_0805_2012Metric_Pad1.15x1.40mm_HandSolder, symbol Device:LED
- added D6: 50% Red, LED_SMD:LED_0805_2012Metric_Pad1.15x1.40mm_HandSolder, symbol Device:LED
- added D7: 75% Red, LED_SMD:LED_0805_2012Metric_Pad1.15x1.40mm_HandSolder, symbol Device:LED
- added D8: 100% Green, LED_SMD:LED_0805_2012Metric_Pad1.15x1.40mm_HandSolder, symbol Device:LED
- added IC1: DW06D, DW06D:DW06D_SFE, symbol DW06D:DW06D
- added J1: Solar_Panel_1, Connector_JST:JST_XH_S2B-XH-A_1x02_P2.50mm_Horizontal, symbol Connector:Conn_01x02_Pin
- added J2: Solar_Panel_2, Connector_JST:JST_XH_S2B-XH-A_1x02_P2.50mm_Horizontal, symbol Connector:Conn_01x02_Pin
- added J3: USBPwrIn, Connector_USB:USB_C_Receptacle_GCT_USB4125-xx-x_6P_TopMnt_Horizontal, symbol Connector:USB_C_Receptacle_PowerOnly_6P
- added J4: Release Detection, Connector_JST:JST_XH_S2B-XH-A_1x02_P2.50mm_Horizontal, symbol Connector:Conn_01x02_Pin
- added L1: 1uH, INDPM7366X300N, symbol MCS0630-100MN1:MCS0630-100MN1
- added R1, R13, R4: 1k5, Resistor_SMD:R_0805_2012Metric_Pad1.20x1.40mm_HandSolder, symbol Device:R
- added R10: 10k, Resistor_SMD:R_0805_2012Metric_Pad1.20x1.40mm_HandSolder, symbol Device:R
- added R2: 7k5, Resistor_SMD:R_0805_2012Metric_Pad1.20x1.40mm_HandSolder, symbol Device:R
- added R3: 30k, Resistor_SMD:R_0805_2012Metric_Pad1.20x1.40mm_HandSolder, symbol Device:R
- added R5, R6: 5k1, Resistor_SMD:R_0805_2012Metric_Pad1.20x1.40mm_HandSolder, symbol Device:R
- added R7: 2R, Resistor_SMD:R_0805_2012Metric_Pad1.20x1.40mm_HandSolder, symbol Device:R
- added R8: 0R5, Resistor_SMD:R_0805_2012Metric_Pad1.20x1.40mm_HandSolder, symbol Device:R
- added S1: USB-Solar Toggle, SS12D10L3, symbol SS-12D10L3:SS-12D10L3
- added S2: Push-Button, PTS647SM50SMTR2LFS, symbol PTS647SM50SMTR2LFS:PTS647SM50SMTR2LFS
- added S3: Power Switch, SS12D10L3, symbol SS-12D10L3:SS-12D10L3
- added U1, U4: ACS712xLCTR-05B, Package_SO:SOIC-8_3.9x4.9mm_P1.27mm, symbol Sensor_Current:ACS712xLCTR-05B
- added U2: IP5306, IP5306:SOIC9P127_490X600X170L84X42T330X241N, symbol IP5306:IP5306
- renumbered BT2 to BT1, BT1 to BT2, C1 to C5, D1 to D9, R2 to R11, R1 to R12, R3 to R9, U2 to U3
Connections:
- net GND: now also C1.2, C10.2, C11.2, C12.2, C2.2, C3.2, C4.2, C6.2, C7.2, C8.2, C9.2, D10.1 (K), D3.1 (K), D4.1 (K), IC1.2 (S1), J1.2 (Pin_2), J2.2 (Pin_2), J3.A12 (GND), J3.B12 (GND), J3.S1 (SHIELD), R3.2, R5.2, R6.2, S2.3, U1.5 (GND), U2.9 (GND), U4.5 (GND)
- net at BT1.P, BT2.P, C5.1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: now also C7.1, IC1.3 (S2), IC1.6 (VSS), L1.2, R8.1, U2.6 (BAT)
- net at R11.1: now also IC1.1 (V-)
- net at C5.2: now also IC1.5 (VDD)
- new net: J3.B5 (CC2), R5.1
- new net: D1.C, D2.C, R1.1, R2.1, U1.1 (IP+), U1.2 (IP+)
- new net: C3.1, R7.2
- new net: D5.1 (K), D6.2 (A), D7.1 (K), D8.2 (A), U2.4 (LED3)
- new net: D5.2 (A), D6.1 (K), U2.2 (LED1)
- new net: D2.A, J2.1 (Pin_1)
- new net: D7.2 (A), D8.1 (K), U2.3 (LED2)
- new net: D4.2 (A), R4.2
- new net: J4.1 (Pin_1), S3.2 (COM)
- new net: D10.2 (A), R13.2
- new net: C1.1, U1.6 (FILTER)
- new net: C6.1, R8.2
- new net: C11.1, U4.6 (FILTER)
- new net: D1.A, J1.1 (Pin_1)
- new net: S3.1 (NC), U4.3 (IP-), U4.4 (IP-)
- new net: J3.A5 (CC1), R6.1
- new net: L1.1, U2.7 (SW)
- new net: S1.1 (NC), U1.3 (IP-), U1.4 (IP-)
- new net: R10.1, U2.5 (KEY)
- new net: R10.2, S2.1
- new net: D3.2 (A), R1.2
- new net: J3.A9 (VBUS), J3.B9 (VBUS), R4.1, S1.3 (NO)
- new net +5V: C12.1, C2.1, J4.2 (Pin_2), R13.1, U1.8 (VCC), U4.8 (VCC)
- new net ANA1: U1.7 (VIOUT)
- new net ANA2: R2.2, R3.1
- new net ANA3: U4.7 (VIOUT)
- new net VIN: C4.1, R7.1, S1.2 (COM), U2.1 (VCC)
- new net VOUT: C10.1, C8.1, C9.1, U2.8 (VOUT), U4.1 (IP+), U4.2 (IP+)
- no-connect marks 0 -> 4
Other:
- moved on the sheet: BT1, BT2, C5, D9, R11, R12, R9, U3

Commit message: More updates
Parts:
- removed BT1, BT2: 1042, Battery_Holder_1:BAT_1042, symbol Battery_Holder_1:1042
- added BT1, BT2: 1043, 1043:BAT_1043, symbol 1043:1043
- added H1, H2, H3, H4: MountingHole, MountingHole:MountingHole_3.2mm_M3, symbol Mechanical:MountingHole
- added J5: Conn_02x20_Odd_Even, Connector_PinSocket_2.54mm:PinSocket_2x20_P2.54mm_Vertical, symbol Connector_Generic:Conn_02x20_Odd_Even
Connections:
- net +5V: now also J4.1 (Pin_1); no longer J4.2 (Pin_2)
- net GND: no longer R9.2
- net +BATT: now reaches C7.1, D9.1 (K), L1.2, R8.1, R9.1, U2.6 (BAT), U3.1 (G)
- net +BATT: now also BT1.P, BT2.P; no longer C5.1, IC1.3 (S2), IC1.6 (VSS), U3.2 (S)
- net at R12.2, U3.3 (D): now also BT1.N, BT2.N
- net at C5.2, IC1.5 (VDD): now also R9.2
- net at S3.2 (COM): now also J4.2 (Pin_2); no longer J4.1 (Pin_1)
- new net: C5.1, IC1.3 (S2), IC1.6 (VSS), U3.2 (S)

Commit message: Updates
Parts:
- added C13: 10u, Capacitor_SMD:C_0805_2012Metric_Pad1.18x1.45mm_HandSolder, symbol Device:C
- added C14: 100n, Capacitor_SMD:C_0805_2012Metric_Pad1.18x1.45mm_HandSolder, symbol Device:C
- added C15, C16: 22u, Capacitor_SMD:C_0805_2012Metric_Pad1.18x1.45mm_HandSolder, symbol Device:C
- added L2: 4.7uH, INDPM7366X300N, symbol MCS0630-100MN1:MCS0630-100MN1
- added U5: AP63203WU, Package_TO_SOT_SMD:TSOT-23-6, symbol Regulator_Switching:AP63203WU
Connections:
- net +5V: now also J5.1 (Pin_1), C13.1, U5.2 (EN), U5.3 (IN)
- net GND: now also C13.2, C15.2, C16.2, U5.4 (GND)
- net +3.3V: now reaches J5.2 (Pin_2)
- net +3.3V: now also C15.1, C16.1, L2.2, U5.1 (FB)
- new net: C14.1, L2.1, U5.5 (SW)
- new net: C14.2, U5.6 (BST)
Other:
- moved on the sheet: D10, J5, R13

Commit message: Updates
Parts:
- L1, L2: footprint INDPM7366X300N -> MCS0630-100MN1:INDPM7366X300N
- S1, S3: footprint SS12D10L3 -> SS-12D10L3:SS12D10L3
Connections:
- net +BATT: now also J5.39 (Pin_39), J5.40 (Pin_40)
- net ANA1: now also J5.38 (Pin_38)
- net ANA2: now also J5.36 (Pin_36)
- net ANA3: now also J5.34 (Pin_34)
- no-connect marks 4 -> 37

Commit message: EPS and OBC done
Connections:
- net +5V: now also J5.38 (Pin_38)
- net ANA1: now also J5.6 (Pin_6); no longer J5.38 (Pin_38)
- net ANA2: now also J5.20 (Pin_20); no longer J5.36 (Pin_36)
- net ANA3: now also J5.8 (Pin_8); no longer J5.34 (Pin_34)
- no-connect marks 37 -> 36
Changed lines of the file:
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@@
 	)
 	(no_connect
+		(at 298.45 241.3)
+	)
+	(no_connect
 		(at 311.15 203.2)
 	)
@@
 	)
 	(no_connect
+		(at 298.45 243.84)
+	)
+	(no_connect
 		(at 298.45 231.14)
 	)
@@
 	)
 	(no_connect
-		(at 298.45 205.74)
-	)
-	(no_connect
 		(at 311.15 233.68)
 	)
@@
 	)
 	(no_connect
-		(at 298.45 208.28)
-	)
-	(no_connect
 		(at 186.69 161.29)
 	)
@@
 	)
 	(no_connect
-		(at 298.45 223.52)
-	)
-	(no_connect
 		(at 311.15 226.06)
 	)
@@
 	(wire
 		(pts
-			(xy 290.83 243.84) (xy 298.45 243.84)
-		)
-		(stroke
-			(width 0)
-			(type default)
-		)
-	)
-	(wire
-		(pts
 			(xy 232.41 218.44) (xy 232.41 224.79)
 		)
@@
 	(wire
 		(pts
+			(xy 290.83 205.74) (xy 298.45 205.74)
+		)
+		(stroke
+			(width 0)
+			(type default)
+		)
+	)
+	(wire
+		(pts
 			(xy 30.48 209.55) (xy 72.39 209.55)
 		)
@@
 	(wire
 		(pts
-			(xy 290.83 241.3) (xy 298.45 241.3)
-		)
-		(stroke
-			(width 0)
-			(type default)
-		)
-	)
-	(wire
-		(pts
 			(xy 118.11 163.83) (xy 118.11 153.67)
 		)
@@
 	(wire
 		(pts
+			(xy 298.45 246.38) (xy 293.37 246.38)
+		)
+		(stroke
+			(width 0)
+			(type default)
+		)
+	)
+	(wire
+		(pts
 			(xy 161.29 161.29) (xy 166.37 161.29)
 		)
@@
 	(wire
 		(pts
+			(xy 290.83 208.28) (xy 298.45 208.28)
+		)
+		(stroke
+			(width 0)
+			(type default)
+		)
+	)
+	(wire
+		(pts
 			(xy 140.97 179.07) (xy 140.97 163.83)
 		)
@@
 	(wire
 		(pts
+			(xy 290.83 223.52) (xy 298.45 223.52)
+		)
+		(stroke
+			(width 0)
+			(type default)
+		)
+	)
+	(wire
+		(pts
 			(xy 181.61 143.51) (xy 181.61 148.59)
 		)
@@
 	(wire
 		(pts
-			(xy 290.83 246.38) (xy 298.45 246.38)
-		)
-		(stroke
-			(width 0)
-			(type default)
-		)
-	)
-	(wire
-		(pts
 			(xy 96.52 163.83) (xy 111.76 163.83)
 		)
@@
 		)
 	)
+	(label "ANA3"
+		(at 290.83 208.28 0)
+		(fields_autoplaced yes)
+		(effects
+			(font
+				(size 1.27 1.27)
+			)
+			(justify left bottom)
+		)
+	)
 	(label "VOUT"
 		(at 30.48 209.55 0)
@@
 		)
 	)
-	(label "ANA3"
-		(at 290.83 241.3 0)
+	(label "ANA2"
+		(at 290.83 223.52 0)
 		(fields_autoplaced yes)
 		(effects
@@
 	)
 	(label "ANA1"
-		(at 290.83 246.38 0)
+		(at 290.83 205.74 0)
 		(fields_autoplaced yes)
 		(effects
@@
 		)
 	)
-	(label "ANA2"
-		(at 290.83 243.84 0)
-		(fields_autoplaced yes)
-		(effects
-			(font
-				(size 1.27 1.27)
-			)
-			(justify left bottom)
-		)
-	)
 	(label "ANA1"
 		(at 246.38 27.94 180)
@@
 					(unit 1)
 				)
+			)
+		)
+	)
+	(symbol
+		(lib_id "power:+5V")
+		(at 293.37 246.38 0)
+		(mirror y)
+		(unit 1)
+		(exclude_from_sim no)
+		(in_bom yes)
+		(on_board yes)
+		(dnp no)
+		(fields_autoplaced yes)
+		(property "Reference" "#PWR039"
+			(at 293.37 250.19 0)
+			(effects
+				(font
+					(size 1.27 1.27)
+				)
+				(hide yes)
+			)
+		)
+		(property "Value" "+5V"
+			(at 293.37 241.3 0)
+			(effects
+				(font
+					(size 1.27 1.27)
+				)
+			)
+		)
+		(property "Footprint" ""
+			(at 293.37 246.38 0)
+			(effects
+				(font
+					(size 1.27 1.27)
+				)
+				(hide yes)
+			)
+		)
+		(property "Datasheet" ""
+			(at 293.37 246.38 0)
+			(effects
+				(font
+					(size 1.27 1.27)
+				)
+				(hide yes)
+			)
+		)
+		(property "Description" "Power symbol creates a global label with name \"+5V\""
+			(at 293.37 246.38 0)
+			(effects
+				(font
+					(size 1.27 1.27)
+				)
+				(hide yes)
+			)
+		)
+		(pin "1"
+		)
+		(instances
+			(project "EPSv3"
+				(path "/2756be33-b8cf-4e5c-b345-72e2144b0e27"
+					(reference "#PWR039")
+					(unit 1)
+				)
